Commit message: Correção dos arquivos de colisão e substituição da tocha

File: kuka_kr90_support/urdf/kr90r2900_extraha_macro.xacro (robot description, xacro)
@@ -155,9 +155,16 @@
     <link name="${prefix}tool0">
       <visual>
-        <origin xyz="0.0216 0 -0.4853" rpy="${DEG2RAD * 180} 0 0"/>
-        <geometry>
-          <mesh filename="package://kuka_kr90_support/meshes/kr90r2900extraHA/visual/tocha_cmt_centro.dae" />
-        </geometry>
-      </visual>
+        <!-- old torch origin xyz="0.0216 0 -0.4853" rpy="${DEG2RAD * 180} 0 0"/-->
+        <origin xyz="0.001 0 -0.4727" rpy="${DEG2RAD * 180} 0 0"/>
+        <geometry>
+          <mesh filename="package://kuka_kr90_support/meshes/kr90r2900extraHA/visual/tocha.dae" />
+        </geometry>
+      </visual>
+      <collision>
+        <origin xyz="0.001 0 -0.4727" rpy="${DEG2RAD * 180} 0 0"/>
+        <geometry>
+          <mesh filename="package://kuka_kr90_support/meshes/kr90r2900extraHA/collision/tocha.stl" />
+        </geometry>
+      </collision>
     </link>
     <!-- END LINKS -->

Commit message: Correction in te torch axis position

File: kuka_kr90_support/urdf/kr90r2900_extraha_macro.xacro (robot description, xacro)
@@ -161,10 +161,10 @@
         </geometry>
       </visual>
-      <collision>
+      <!--collision>
         <origin xyz="0.001 0 -0.4727" rpy="${DEG2RAD * 180} 0 0"/>
         <geometry>
           <mesh filename="package://kuka_kr90_support/meshes/kr90r2900extraHA/collision/tocha.stl" />
         </geometry>
-      </collision>
+      </collision-->
     </link>
     <!-- END LINKS -->
@@ -222,5 +222,5 @@
       <parent link="${prefix}link_6"/>
       <child link="${prefix}tool0"/>
-      <origin xyz="0.4853 0 0.0216" rpy="0 ${DEG2RAD * 90} 0"/>
+      <origin xyz="0.4727 0 0.001" rpy="0 ${DEG2RAD * 90} 0"/>
       <axis xyz="0 0 -1"/>
     </joint>
